File: HW5/hw5.kicad_sch (KiCad schematic)
At the start: 8 parts, among them J1 Power terminal, J2 Detector_Terminal, Q1 IRFZ44

Commit message: HW4, HW5 complete
Parts:
- BZ1: footprint (none) -> Buzzer_Beeper:Buzzer_12x9.5RM7.6
- J1, LA1: footprint (none) -> TerminalBlock_RND:TerminalBlock_RND_205-00287_1x02_P5.08mm_Horizontal
- J2: value Detector_Terminal -> Detector terminal; footprint (none) -> TerminalBlock_RND:TerminalBlock_RND_205-00287_1x02_P5.08mm_Horizontal
- Q1: footprint (none) -> Package_TO_SOT_THT:TO-220-3_Vertical
- R1, R2: value 330 -> 220; footprint (none) -> Resistor_THT:R_Axial_DIN0207_L6.3mm_D2.5mm_P10.16mm_Horizontal
- R3: value 220К -> 110К; footprint (none) -> Resistor_THT:R_Axial_DIN0207_L6.3mm_D2.5mm_P10.16mm_Horizontal
Connections:
- net +12V: now also J1.1 (Pin_1), J2.2 (Pin_2); no longer J1.2 (Pin_2), J2.1 (Pin_1)
- net GND: now also J1.2 (Pin_2); no longer J1.1 (Pin_1)
- net +12V_COM: now reaches Q1.1 (G), R3.1
- net +12V_COM: now also J2.1 (Pin_1); no longer J2.2 (Pin_2)
- net GND_COM: now reaches LA1.1 (-), Q1.2 (D), R1.1
- net BUZ-: now reaches BZ1.2 (-), R1.2, R2.2
Other:
- moved on the sheet: J1, J2
