File: HW7/hw7/hw7.kicad_sch (KiCad schematic)
At the start: 13 parts, among them J1 Conn_01x02_Pin, J2 Conn_01x02_Socket, J3 Jack-DC, J4 Screw_Terminal_01x02, K1 SANYOU_SRD_Form_C, Q1 BC337-40, U1 817C

Commit message: hw7 proceeding
Parts:
- removed J2: Conn_01x02_Socket, symbol Connector:Conn_01x02_Socket
- added H1, H2, H3, H4: MountingHole, MountingHole:MountingHole_2.2mm_M2_DIN965_Pad, symbol Mechanical:MountingHole
- D1: footprint (none) -> Diode_SMD:D_0805_2012Metric
- D2, D3: footprint (none) -> LED_SMD:LED_1210_3225Metric
- J1: renamed from J3; footprint (none) -> Connector_BarrelJack:BarrelJack_GCT_DCJ200-10-A_Horizontal
- J2: renamed from J1; footprint (none) -> Connector_Molex:Molex_PicoBlade_53261-0271_1x02-1MP_P1.25mm_Horizontal
- J3: renamed from J4; footprint (none) -> TerminalBlock_Phoenix:TerminalBlock_Phoenix_MKDS-1,5-2-5.08_1x02_P5.08mm_Horizontal
- Q1: footprint (none) -> Package_TO_SOT_THT:TO-92L
- R1, R2, R3: footprint (none) -> Resistor_SMD:R_0805_2012Metric_Pad1.20x1.40mm_HandSolder
- U1: footprint (none) -> Package_DIP:DIP-4_W7.62mm_LongPads
Connections:
- net GND: now also J3.2 (Pin_2)
- net GNDS: now also J2.2 (Pin_2), U1.2
- net VS: now also J2.1 (Pin_1), R2.1
- net +5V: now reaches D1.1 (K), J1.1, K1.1, K1.2, R3.1
Other:
- moved on the sheet: D3, J3

Commit message: HW7-HW8
Parts:
- added J4: Conn_01x02_Pin, Connector_Molex:Molex_KK-254_AE-6410-02A_1x02_P2.54mm_Vertical, symbol Connector:Conn_01x02_Pin
- added R4: 10к, Resistor_SMD:R_0805_2012Metric_Pad1.20x1.40mm_HandSolder, symbol Device:R
- added R5: 510, Resistor_SMD:R_0805_2012Metric_Pad1.20x1.40mm_HandSolder, symbol Device:R
- added U2: 817C, Package_DIP:DIP-4_W7.62mm_LongPads, symbol Isolator:Optocoupler_DC_PhotoNPN_AKEC
- H1, H2, H3, H4: symbol Mechanical:MountingHole -> Mechanical:MountingHole_Pad
- J2: footprint Connector_Molex:Molex_PicoBlade_53261-0271_1x02-1MP_P1.25mm_Horizontal -> Connector_Molex:Molex_KK-254_AE-6410-02A_1x02_P2.54mm_Vertical
- LED1: renamed from D3; value Green -> Red
- LED2: renamed from D2; value Red -> Green
Connections:
- net GND: now also H1.1, H2.1, H3.1, H4.1, R4.2
- net GNDS: now also J4.2 (Pin_2), U2.2
- net at Q1.2 (B), U1.3: now also R4.1
- net +5V renamed +12V
- net VS renamed VS2
- new net: R5.2, U2.1
- new net VS1: J4.1 (Pin_1), R5.1
Other:
- moved on the sheet: LED1, R3

Commit message: HW7 done, HW8 processing
Parts:
- removed J4: Conn_01x02_Pin, Connector_Molex:Molex_KK-254_AE-6410-02A_1x02_P2.54mm_Vertical, symbol Connector:Conn_01x02_Pin
- removed R5: 510, Resistor_SMD:R_0805_2012Metric_Pad1.20x1.40mm_HandSolder, symbol Device:R
- removed U2: 817C, Package_DIP:DIP-4_W7.62mm_LongPads, symbol Isolator:Optocoupler_DC_PhotoNPN_AKEC
Connections:
- net +12V renamed +5V
