File: HW9/hw9/hw9.kicad_pcb (KiCad board)
At the start: 2 copper layers, 52.7 x 33.7 mm, 33 parts, among them J1 Barrel_Jack_MountingPin, Q1 BC337, SW1 SW_MEC_5G, U1 LM317, U2 NE555P, U3 NE555P

Commit message: hw9 done
Parts:
- added H5: MountingHole_Pad, MountingHole:MountingHole_2.2mm_M2_DIN965_Pad, F.Cu at (50.0, 59.4)
- added J2: Conn_01x02_Pin, Connector_Molex:Molex_PicoBlade_53261-0271_1x02-1MP_P1.25mm_Horizontal, F.Cu at (67.0, 77.5)
- moved H2 34.9 mm to (20.6, 71.6)
- moved H3 16.1 mm to (67.6, 59.4)
- moved H4 11.2 mm to (61.0, 80.6)
- moved R10 6.37 mm to (68.6, 85.9), turned to 90 degrees
- moved R4 6.02 mm to (57.8, 85.7), turned to 90 degrees
- moved C6 2.64 mm to (49.3, 72.4)
- moved R7 2.19 mm to (56.5, 58.4)
- moved R8 2.05 mm to (47.8, 65.4)
- moved D3 1.90 mm to (61.0, 86.5)
- moved R9 1.55 mm to (62.2, 58.4), turned to 180 degrees
- moved C1 1.52 mm to (26.0, 70.5)
- moved D4 1.51 mm to (65.5, 86.5), turned to -90 degrees
- moved D1 1.18 mm to (29.8, 63.6)
- moved R1 1.17 mm to (24.8, 63.6)
- moved R2 1.11 mm to (24.8, 66.2)
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Routing:
- net Net-(J2-Pin_2): track 11.1 -> 19.6 mm
- net GND: track 11.2 -> 18.1 mm
- net Net-(SW1-B): track 40.5 -> 45.7 mm
- net Net-(D4-K): track 30.5 -> 27.6 mm
- net Net-(U3-DISCH): track 4.04 -> 6.53 mm
- net Net-(Q1-B): track 7.68 -> 5.22 mm
- net +12V: track 24.6 -> 22.2 mm
- net CTRL: track 39.2 -> 41.0 mm
- net Net-(D2-A): track 16.5 -> 15.1 mm
- net +9V: track 109.8 -> 110.9 mm
- net Net-(D3-A): track 4.01 -> 5.07 mm
Other:
- board text added: "D4"
