File: HW8/hw8/hw8.kicad_sch (KiCad schematic)
At the start: 0 parts

Commit message: HW7 done, HW8 processing
Parts:
- added C1: 0.1uF, symbol Device:C
- added C2, C3: 10uF, symbol Device:C_Polarized
- added D1, D2: 1N4007, symbol Device:D
- added D3, D4: 1N4007, Diode_THT:D_DO-41_SOD81_P10.16mm_Horizontal, symbol Diode:1N4007
- added J1: Barrel_Jack, symbol Connector:Barrel_Jack
- added J2, J4: Conn_01x02_Pin, symbol Connector:Conn_01x02_Pin
- added J3: Comm 1 Terminal, symbol Connector:Screw_Terminal_01x03
- added J5: Comm 2 Terminal, symbol Connector:Screw_Terminal_01x03
- added K1, K2: SANYOU_SRD_Form_C, Relay_THT:Relay_SPDT_SANYOU_SRD_Series_Form_C, symbol Relay:SANYOU_SRD_Form_C
- added Q1, Q2: BC337, Package_TO_SOT_THT:TO-92_Inline, symbol Transistor_BJT:BC337
- added R1: 240, symbol Device:R
- added R2: 720, symbol Device:R
- added R3, R4: 2k, symbol Device:R
- added U1: LM317_TO-220, Package_TO_SOT_THT:TO-220-3_Vertical, symbol Regulator_Linear:LM317_TO-220
- added U2, U3: PC817, Package_DIP:DIP-4_W7.62mm, symbol Isolator:PC817
Connections:
- new net: J3.1 (Pin_1), K1.4
- new net: J3.2 (Pin_2), K1.3
- new net: J3.3 (Pin_3), K1.1
- new net: D4.2 (A), K2.2, Q1.1 (C)
- new net: Q1.2 (B), U3.3
- new net: C2.1, D1.2 (A), R1.2, R2.2, U1.1 (ADJ)
- new net: D3.2 (A), K1.2, Q2.1 (C)
- new net: R3.2, U2.1
- new net: Q2.2 (B), U2.3
- new net: J5.3 (Pin_3), K2.1
- new net: J5.2 (Pin_2), K2.3
- new net: J5.1 (Pin_1), K2.4
- new net: R4.2, U3.1
- new net +12V: C1.1, D2.1 (K), J1.1, U1.3 (VI)
- new net +5V: C3.1, D1.1 (K), D2.2 (A), D3.1 (K), D4.1 (K), K1.5, K2.5, R1.1, U1.2 (VO), U2.4, U3.4
- new net GND: C1.2, C2.2, C3.2, J1.2, Q1.3 (E), Q2.3 (E), R2.1
- new net GNDS: J2.2 (Pin_2), J4.2 (Pin_2), U2.2, U3.2
- new net VS1: J2.1 (Pin_1), R3.1
- new net VS2: J4.1 (Pin_1), R4.1

Commit message: hw8 processing
Parts:
- added H1, H2, H3, H4: MountingHole_Pad, MountingHole:MountingHole_2.2mm_M2_DIN965_Pad, symbol Mechanical:MountingHole_Pad
- C1: footprint (none) -> Capacitor_SMD:C_1206_3216Metric_Pad1.33x1.80mm_HandSolder
- C2, C3: footprint (none) -> Capacitor_THT:CP_Radial_D4.0mm_P1.50mm
- D1, D2: footprint (none) -> Diode_SMD:D_1206_3216Metric
- D3, D4: footprint Diode_THT:D_DO-41_SOD81_P10.16mm_Horizontal -> Diode_SMD:D_1206_3216Metric
- J1: footprint (none) -> Connector_BarrelJack:BarrelJack_GCT_DCJ200-10-A_Horizontal
- J2, J4: footprint (none) -> Connector_Molex:Molex_KK-254_AE-6410-02A_1x02_P2.54mm_Vertical
- J3, J5: footprint (none) -> TerminalBlock_Phoenix:TerminalBlock_Phoenix_MKDS-1,5-3-5.08_1x03_P5.08mm_Horizontal
- R1, R2, R3, R4: footprint (none) -> Resistor_SMD:R_1206_3216Metric_Pad1.30x1.75mm_HandSolder
Connections:
- net GND: now also H1.1, H2.1, H3.1, H4.1

Commit message: hw9 done
Connections:
- net at J3.1 (Pin_1): now also K1.3; no longer K1.4
- net at J3.2 (Pin_2): now also K1.4; no longer K1.3
- net at K2.3: now also J5.1 (Pin_1); no longer J5.2 (Pin_2)
- net at K2.4: now also J5.2 (Pin_2); no longer J5.1 (Pin_1)
Changed lines of the file:
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@@
 	(wire
 		(pts
-			(xy 113.03 124.46) (xy 116.84 124.46)
+			(xy 116.84 116.84) (xy 116.84 121.92)
 		)
 		(stroke
@@
 	(wire
 		(pts
-			(xy 116.84 77.47) (xy 116.84 85.09)
-		)
-		(stroke
-			(width 0)
-			(type default)
-		)
-	)
-	(wire
-		(pts
 			(xy 54.61 53.34) (xy 54.61 60.96)
 		)
@@
 	(wire
 		(pts
-			(xy 102.87 114.3) (xy 116.84 114.3)
+			(xy 102.87 114.3) (xy 113.03 114.3)
 		)
 		(stroke
@@
 	(wire
 		(pts
-			(xy 116.84 114.3) (xy 116.84 121.92)
-		)
-		(stroke
-			(width 0)
-			(type default)
-		)
-	)
-	(wire
-		(pts
 			(xy 160.02 106.68) (xy 160.02 118.11)
 		)
@@
 	(wire
 		(pts
-			(xy 107.95 80.01) (xy 113.03 80.01)
+			(xy 107.95 80.01) (xy 116.84 80.01)
 		)
 		(stroke
@@
 	(wire
 		(pts
-			(xy 113.03 80.01) (xy 113.03 87.63)
+			(xy 116.84 80.01) (xy 116.84 85.09)
 		)
 		(stroke
@@
 	(wire
 		(pts
-			(xy 102.87 77.47) (xy 116.84 77.47)
+			(xy 102.87 77.47) (xy 113.03 77.47)
 		)
 		(stroke
@@
 	(wire
 		(pts
+			(xy 116.84 87.63) (xy 113.03 87.63)
+		)
+		(stroke
+			(width 0)
+			(type default)
+		)
+	)
+	(wire
+		(pts
 			(xy 48.26 85.09) (xy 54.61 85.09)
 		)
@@
 	(wire
 		(pts
+			(xy 107.95 116.84) (xy 116.84 116.84)
+		)
+		(stroke
+			(width 0)
+			(type default)
+		)
+	)
+	(wire
+		(pts
 			(xy 87.63 100.33) (xy 77.47 100.33)
 		)
@@
 	(wire
 		(pts
-			(xy 113.03 116.84) (xy 113.03 124.46)
-		)
-		(stroke
-			(width 0)
-			(type default)
-		)
-	)
-	(wire
-		(pts
 			(xy 101.6 60.96) (xy 113.03 60.96)
 		)
@@
 	(wire
 		(pts
+			(xy 113.03 114.3) (xy 113.03 124.46)
+		)
+		(stroke
+			(width 0)
+			(type default)
+		)
+	)
+	(wire
+		(pts
 			(xy 83.82 80.01) (xy 95.25 80.01)
 		)
@@
 	(wire
 		(pts
-			(xy 113.03 87.63) (xy 116.84 87.63)
-		)
-		(stroke
-			(width 0)
-			(type default)
-		)
-	)
-	(wire
-		(pts
 			(xy 105.41 95.25) (xy 113.03 95.25)
 		)
@@
 	(wire
 		(pts
+			(xy 116.84 124.46) (xy 113.03 124.46)
+		)
+		(stroke
+			(width 0)
+			(type default)
+		)
+	)
+	(wire
+		(pts
 			(xy 82.55 60.96) (xy 91.44 60.96)
 		)
@@
 	(wire
 		(pts
-			(xy 107.95 116.84) (xy 113.03 116.84)
-		)
-		(stroke
-			(width 0)
-			(type default)
-		)
-	)
-	(wire
-		(pts
 			(xy 54.61 129.54) (xy 54.61 132.08)
 		)
@@
 		)
 		(stroke
+			(width 0)
+			(type default)
+		)
+	)
+	(wire
+		(pts
+			(xy 113.03 87.63) (xy 113.03 77.47)
+		)
+		(stroke

Commit message: hw8 processing, hw9 done
Parts:
- added LED1, LED2: LED, LED_SMD:LED_1206_3216Metric, symbol Device:LED
- added R4, R6: 1k, Resistor_SMD:R_1206_3216Metric_Pad1.30x1.75mm_HandSolder, symbol Device:R
- R1: value 240 -> 220
- R2: value 720 -> 680
- renumbered C3 to C2, C2 to C3, D2 to D1, D1 to D2, J3 to J2, J2 to J3, J5 to J4, J4 to J5, Q2 to Q1, Q1 to Q2, R4 to R5
Connections:
- net +5V: now also LED1.2 (A), LED2.2 (A)
- net at D4.2 (A), K2.2, Q2.1 (C): now also R6.1
- net at D3.2 (A), K1.2, Q1.1 (C): now also R4.1
- new net: LED1.1 (K), R4.2
- new net: LED2.1 (K), R6.2
Other:
- note added: "Channel 1"
- note added: "Channel 2"
- note added: "Power source"
- moved on the sheet: D3, D4
