File: HW10/hw10/hw10.kicad_pcb (KiCad board)
At the start: 2 copper layers, 52.5 x 46 mm, 28 parts, among them J1 Screw_Terminal_01x02, J2 Screw_Terminal_01x02, Q1 BC807, Q2 BC817, Q3 IRLZ44N, U1 LM317_TO-220, U2 NE555P

Commit message: HW10 circuit done
Parts:
- added LED1: LED, LED_SMD:LED_1206_3216Metric_Pad1.42x1.75mm_HandSolder, F.Cu at (120.0, 51.4)
- added R7: 22, Resistor_SMD:R_1206_3216Metric_Pad1.30x1.75mm_HandSolder, F.Cu at (132.1, 57.1)
- C3: value 0.1u -> 1.0u
- R4: value 100 -> 200
- R5: value 150 -> 1k
- R6: value 30 -> 22
- moved R5 11.4 mm to (120.0, 54.6)
- moved R6 6.40 mm to (125.7, 57.1), turned to 0 degrees
- moved Q1 4.04 mm to (132.1, 62.5)
- moved Q2 4.04 mm to (125.7, 62.5)
- moved R4 3.18 mm to (121.3, 62.9), turned to 90 degrees
- turned C3 to 90 degrees
- turned D3 to 90 degrees
- turned D4 to 90 degrees
Connections:
- C3 pad 1: GND -> +5V
- C3 pad 2: +5V -> GND
- C4 pad 1: Net-(D4-K) -> Net-(D4-A)
- Q1 pad 2: +12V -> Net-(Q1-E)
- Q2 pad 1: Net-(Q2-B) -> Net-(Q1-B)
- Q2 pad 2: GND -> Net-(Q1-E)
- Q2 pad 3: Net-(Q1-C) -> Net-(Q2-C)
- Q3 pad 1: Net-(Q3-G) -> Net-(Q1-E)
- R4 pad 1: Net-(Q2-B) -> Net-(Q1-B)
- R5 pad 1: Net-(Q1-B) -> Net-(LED1-A)
- R5 pad 2: Net-(Q2-B) -> Net-(U2-OUT)
- R6 pad 1: Net-(Q3-G) -> +12V
- R6 pad 2: Net-(Q1-C) -> Net-(Q2-C)
- RV1 pad 1: Net-(D3-A) -> Net-(D3-K)
- RV1 pad 2: Net-(D4-K) -> Net-(D4-A)
- RV1 pad 3: Net-(D4-K) -> Net-(D4-A)
- RV2 pad 1: Net-(D3-K) -> Net-(D3-A)
- RV2 pad 3: Net-(D4-A) -> Net-(D4-K)
- U2 pad 2: Net-(D4-K) -> Net-(D4-A)
- U2 pad 6: Net-(D4-K) -> Net-(D4-A)
Routing:
- net Net-(D4-K): track 44.1 -> 12.5 mm
- net Net-(D4-A): track 12.5 -> 44.1 mm
- net Net-(Q1-E): track 0.00 -> 20.4 mm
- net Net-(Q2-B): track 9.21 -> 0.00 mm
- net Net-(Q1-C): track 12.6 -> 4.86 mm
- net Net-(D3-K): track 10.3 -> 18.0 mm
- net Net-(D3-A): track 18.0 -> 10.3 mm
- net Net-(U2-OUT): track 20.6 -> 27.8 mm, vias 1 -> 2
- net Net-(Q1-B): track 7.34 -> 13.2 mm
- net Net-(Q2-C): track 0.00 -> 4.86 mm
- net Net-(Q3-G): track 4.63 -> 0.00 mm
- net Net-(D2-A): track 36.6 -> 32.8 mm
- net Net-(LED1-A): track 0.00 -> 3.20 mm
- net GND: track 21.3 -> 23.0 mm, vias 4 -> 5
- net +12V: track 103.3 -> 102.5 mm

Commit message: HW10 done
Connections:
- net Net-(U2-OUT) renamed PWM
Changed lines of the file:
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@@
 	(net 14 "Net-(Q1-E)")
 	(net 15 "Net-(U2-DISCH)")
-	(net 16 "Net-(U2-OUT)")
+	(net 16 "PWM")
 	(net 17 "Net-(Q2-C)")
 	(footprint "Package_DIP:DIP-8_W7.62mm"
@@
 			(layers "*.Cu" "*.Mask")
 			(remove_unused_layers no)
-			(net 16 "Net-(U2-OUT)")
+			(net 16 "PWM")
 			(pinfunction "OUT")
 			(pintype "output")
@@
 			)
 		)
-		(property "Datasheet" ""
+		(property "Datasheet" "~"
 			(at 0 0 0)
 			(layer "F.Fab")
@@
 			)
 		)
-		(property "Datasheet" ""
+		(property "Datasheet" "~"
 			(at 0 0 270)
 			(unlocked yes)
@@
 			)
 		)
-		(property "Datasheet" ""
+		(property "Datasheet" "~"
 			(at 0 0 90)
 			(layer "F.Fab")
@@
 			)
 		)
-		(property "Datasheet" ""
+		(property "Datasheet" "~"
 			(at 0 0 270)
 			(unlocked yes)
@@
 			)
 		)
-		(property "Datasheet" ""
+		(property "Datasheet" "~"
 			(at 0 0 90)
 			(layer "F.Fab")
@@
 			)
 		)
-		(property "Datasheet" ""
+		(property "Datasheet" "~"
 			(at 0 0 0)
 			(layer "F.Fab")
@@
 			)
 		)
-		(property "Datasheet" ""
+		(property "Datasheet" "~"
 			(at 0 0 90)
 			(layer "F.Fab")
@@
 			(layers "F.Cu" "F.Mask" "F.Paste")
 			(roundrect_rratio 0.192308)
-			(net 16 "Net-(U2-OUT)")
+			(net 16 "PWM")
 			(pintype "passive")
 		)
@@
 			)
 		)
-		(property "Datasheet" ""
+		(property "Datasheet" "~"
 			(at 0 0 0)
 			(layer "F.Fab")
@@
 			)
 		)
-		(property "Datasheet" ""
+		(property "Datasheet" "~"
 			(at 0 0 0)
 			(layer "F.Fab")
@@
 			)
 		)
-		(property "Datasheet" ""
+		(property "Datasheet" "~"
 			(at 0 0 0)
 			(layer "F.Fab")
@@
 			)
 		)
-		(property "Datasheet" ""
+		(property "Datasheet" "~"
 			(at 0 0 0)
 			(layer "F.Fab")
@@
 			)
 		)
-		(property "Datasheet" ""
+		(property "Datasheet" "~"
 			(at 0 0 0)
 			(layer "F.Fab")
@@
 			(layers "F.Cu" "F.Mask" "F.Paste")
 			(roundrect_rratio 0.192308)
-			(net 16 "Net-(U2-OUT)")
+			(net 16 "PWM")
 			(pintype "passive")
 		)
@@
 			)
 		)
-		(property "Datasheet" ""
+		(property "Datasheet" "~"
 			(at 0 0 0)
 			(layer "F.Fab")
@@
 			)
 		)
-		(property "Datasheet" ""
+		(property "Datasheet" "~"
 			(at 0 0 0)
 			(layer "F.Fab")
@@
 			)
 		)
-		(property "Datasheet" ""
+		(property "Datasheet" "~"
 			(at 0 0 90)
 			(layer "F.Fab")
@@
 			)
 		)
-		(property "Datasheet" ""
+		(property "Datasheet" "~"
 			(at 0 0 0)
 			(layer "F.Fab")
@@
 			)
 		)
-		(property "Datasheet" ""
+		(property "Datasheet" "~"
 			(at 0 0 90)
 			(layer "F.Fab")
@@
 			)
 		)
-		(property "Datasheet" ""
+		(property "Datasheet" "~"
 			(at 0 0 0)
 			(layer "F.Fab")
@@
 			)
 		)
-		(property "Datasheet" ""
+		(property "Datasheet" "~"
 			(at 0 0 90)
 			(layer "F.Fab")
@@
 			)
 		)
-		(property "Datasheet" ""
+		(property "Datasheet" "~"
 			(at 0 0 0)
 			(layer "F.Fab")
@@
 			)
 		)
-		(property "Datasheet" ""
+		(property "Datasheet" "~"
 			(at 0 0 0)
 			(layer "F.Fab")
