File: HW10/hw10/hw10.kicad_sch (KiCad schematic)
At the start: 0 parts

Commit message: HW10 processing
Parts:
- added C1, C3: 0.1u, Capacitor_SMD:C_1206_3216Metric_Pad1.33x1.80mm_HandSolder, symbol Device:C
- added C2: 10u, Capacitor_THT:CP_Radial_D4.0mm_P1.50mm, symbol Device:C_Polarized
- added C4: 1u, Capacitor_THT:CP_Radial_D4.0mm_P1.50mm, symbol Device:C
- added C5: 0.01u, Capacitor_SMD:C_1206_3216Metric_Pad1.33x1.80mm_HandSolder, symbol Device:C
- added D1, D2, D3, D4: 1N4007, Diode_SMD:D_SMA_Handsoldering, symbol Diode:1N4007
- added H1, H2, H3, H4: MountingHole_Pad, MountingHole:MountingHole_2.2mm_M2_DIN965_Pad, symbol Mechanical:MountingHole_Pad
- added J1, J2: Screw_Terminal_01x02, TerminalBlock_Phoenix:TerminalBlock_Phoenix_MKDS-1,5-2-5.08_1x02_P5.08mm_Horizontal, symbol Connector:Screw_Terminal_01x02
- added Q1: BC807, Package_TO_SOT_SMD:SOT-23_Handsoldering, symbol Transistor_BJT:BC807
- added Q2: BC817, Package_TO_SOT_SMD:SOT-23_Handsoldering, symbol Transistor_BJT:BC817
- added Q3: IRLZ44N, Package_TO_SOT_THT:TO-220-3_Vertical, symbol Transistor_FET:IRLZ44N
- added R1: 680, Resistor_SMD:R_1206_3216Metric_Pad1.30x1.75mm_HandSolder, symbol Device:R
- added R2: 220, Resistor_SMD:R_1206_3216Metric_Pad1.30x1.75mm_HandSolder, symbol Device:R
- added R3: 1k, Resistor_SMD:R_1206_3216Metric_Pad1.30x1.75mm_HandSolder, symbol Device:R
- added R4: 100, Resistor_SMD:R_1206_3216Metric_Pad1.30x1.75mm_HandSolder, symbol Device:R
- added R5: 150, Resistor_SMD:R_1206_3216Metric_Pad1.30x1.75mm_HandSolder, symbol Device:R
- added R6: 30, Resistor_SMD:R_1206_3216Metric_Pad1.30x1.75mm_HandSolder, symbol Device:R
- added RV1, RV2: 50k, Potentiometer_THT:Potentiometer_Alps_RK09K_Single_Vertical, symbol Device:R_Potentiometer
- added U1: LM317_TO-220, Package_TO_SOT_THT:TO-220-3_Vertical, symbol Regulator_Linear:LM317_TO-220
- added U2: NE555P, Package_DIP:DIP-8_W7.62mm, symbol Timer:NE555P
Connections:
- new net: C4.1, D4.1 (K), RV1.2, RV1.3, U2.2 (TRIG), U2.6 (THRES)
- new net: C5.2, U2.5 (CONT)
- new net: Q2.1 (B), R4.1, R5.2
- new net: R4.2, U2.3 (OUT)
- new net: D3.1 (K), RV2.1
- new net: D3.2 (A), RV1.1
- new net: Q1.1 (B), R5.1
- new net: Q1.3 (C), Q2.3 (C), R6.2
- new net: Q3.1 (G), R6.1
- new net: C2.1, D2.2 (A), R1.1, R2.1, U1.1 (ADJ)
- new net: J2.2 (Pin_2), Q3.2 (D)
- new net: R3.1, RV2.2, U2.7 (DISCH)
- new net: D4.2 (A), RV2.3
- new net +12V: C1.2, D1.1 (K), J1.1 (Pin_1), J2.1 (Pin_1), Q1.2 (E), U1.3 (VI)
- new net +5V: C3.2, D1.2 (A), D2.1 (K), R2.2, R3.2, U1.2 (VO), U2.4 (~{RST}), U2.8 (VCC)
- new net GND: C1.1, C2.2, C3.1, C4.2, C5.1, H1.1, H2.1, H3.1, H4.1, J1.2 (Pin_2), Q2.2 (E), Q3.3 (S), R1.2, U2.1 (GND)

Commit message: HW10 circuit done
Parts:
- added LED1: LED, LED_SMD:LED_1206_3216Metric_Pad1.42x1.75mm_HandSolder, symbol Device:LED
- added R7: 22, Resistor_SMD:R_1206_3216Metric_Pad1.30x1.75mm_HandSolder, symbol Device:R
- C3: value 0.1u -> 1.0u; symbol Device:C -> Device:C_Polarized
- C4: symbol Device:C -> Device:C_Polarized
- R4: value 100 -> 200
- R5: value 150 -> 1k
- R6: value 30 -> 22
Connections:
- net +12V: now also R6.1; no longer Q1.2 (E)
- net +5V: now also C3.1; no longer C3.2
- net GND: now also C3.2, LED1.1 (K), R7.2; no longer C3.1, Q2.2 (E)
- net at C4.1, RV1.2, RV1.3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: now also D4.2 (A); no longer D4.1 (K)
- net at Q2.1 (B), R4.1: now also Q1.1 (B); no longer R5.2
- net at R4.2, U2.3 (OUT): now also R5.2
- net at D3.1 (K): now also RV1.1; no longer RV2.1
- net at D3.2 (A): now also RV2.1; no longer RV1.1
- net at R5.1: now also LED1.2 (A); no longer Q1.1 (B)
- net at Q2.3 (C), R6.2: no longer Q1.3 (C)
- net at Q3.1 (G): now also Q1.2 (E), Q2.2 (E); no longer R6.1
- net at RV2.3: now also D4.1 (K); no longer D4.2 (A)
- new net: Q1.3 (C), R7.1
Other:
- moved on the sheet: D3, D4, J2, Q1, Q2, Q3

Commit message: HW10 done
Connections:
- net PWM: now reaches R4.2, R5.2, U2.3 (OUT)
Other:
- moved on the sheet: C1, C2, C3, C4, C5, D1, D2, D3, D4, J1, J2, LED1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
