File: HW11/HW11/HW11.kicad_sch (KiCad schematic)
At the start: 16 parts

Commit message: HW13 started
Parts:
- removed C?: C, symbol Device:C
- removed L?: L, symbol Device:L
- added C1: 100u, Capacitor_THT:CP_Radial_D4.0mm_P1.50mm, symbol Device:C_Polarized
- added H1, H2, H3, H4: MountingHole_Pad, MountingHole:MountingHole_2.2mm_M2_Pad, symbol Mechanical:MountingHole_Pad
- added J2: Conn_01x02_Pin, Connector_Phoenix_GMSTB:PhoenixContact_GMSTBVA_2,5_2-G_1x02_P7.50mm_Vertical, symbol Connector:Conn_01x02_Pin
- C2: renamed from C?; value C -> 1nF; footprint (none) -> Capacitor_SMD:C_1206_3216Metric_Pad1.33x1.80mm_HandSolder
- C3: renamed from C?; value C_Polarized -> 220u; footprint (none) -> Capacitor_THT:CP_Radial_D4.0mm_P1.50mm
- D1: renamed from D?; value D_Schottky -> 1N5819; footprint (none) -> Diode_SMD:D_SMB_Handsoldering
- J1: renamed from J?; footprint (none) -> Connector_Phoenix_GMSTB:PhoenixContact_GMSTBVA_2,5_2-G_1x02_P7.50mm_Vertical
- L1: renamed from L?; value L -> 330; footprint (none) -> Inductor_SMD:L_Coilcraft_MSS1260-XXX
- LED1: renamed from LED?; footprint (none) -> LED_SMD:LED_1206_3216Metric
- R1: renamed from R?; value R -> 1k; footprint (none) -> Resistor_SMD:R_1206_3216Metric_Pad1.30x1.75mm_HandSolder
- R2: renamed from R?; value R -> 0.22; footprint (none) -> Resistor_SMD:R_1206_3216Metric_Pad1.30x1.75mm_HandSolder
- R3: renamed from R?; value R -> 2k2; footprint (none) -> Resistor_SMD:R_1206_3216Metric_Pad1.30x1.75mm_HandSolder
- R4: renamed from R?; value R -> 67; footprint (none) -> Resistor_SMD:R_1206_3216Metric_Pad1.30x1.75mm_HandSolder
- R5: renamed from R?; value R -> 5k; footprint (none) -> Resistor_SMD:R_1206_3216Metric_Pad1.30x1.75mm_HandSolder
- R6: renamed from R?; value R -> 68k; footprint (none) -> Resistor_SMD:R_1206_3216Metric_Pad1.30x1.75mm_HandSolder
- RV1: renamed from RV?; value 50k -> 100k; footprint (none) -> Potentiometer_THT:Potentiometer_Bourns_3296Y_Vertical
- gave numbers to parts that had none: 1
Connections:
- net +5V: now also C1.1
- net GND: now also C1.2, H1.1, H2.1, H3.1, H4.1, J2.2 (Pin_2); no longer R6.1, RV1.1, RV1.2
- net at R3.2, U1.5 (Vfb): now also R5.2; no longer R5.1
- net at C3.1, D1.1 (K), R6.2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: now also J2.1 (Pin_1); no longer R5.2
- new net: R5.1, R6.1, RV1.1, RV1.2
Other:
- moved on the sheet: C2, C3, D1, J1, LED1, R1, R5, R6, RV1
