File: HW12/HW12/HW12.kicad_pcb (KiCad board)
At the start: 2 copper layers, 110.5 x 39 mm, 68 parts, among them J1 Barrel_Jack_MountingPin, Q1 BC337, U1 MC34063AP, U2 LM7805_TO220, U3 NE555P, U4 74HC595, U5 74HC595, U6 74HC595

Commit message: hw12 corr
Parts:
- removed U5: 74HC595, Package_DIP:DIP-16_W7.62mm
Connections:
- R10 pad 1: Net-(Q1-C) -> +5V
- R10 pad 2: +5V -> Net-(Q1-C)
- R17 pad 1: Net-(U5-QA) -> Net-(Q1-B)
- R17 pad 2: Net-(Q1-B) -> Net-(U6-QH)
- R18 pad 1: Net-(U5-SER) -> Net-(U6-QH)
- U4 pad 9: unconnected-(U4-QH'-Pad9) -> Net-(U4-QH')
- U6 pad 14: Net-(U4-QH) -> Net-(U4-QH')
- U6 pad 7: Net-(U5-SER) -> Net-(U6-QH)
Routing:
- net Net-(U6-QH): track 0.00 -> 40.8 mm
- net Net-(U5-SER): track 40.8 -> 0.00 mm
- net Net-(U5-QA): track 24.2 -> 0.00 mm
- net Net-(Q1-B): track 3.59 -> 27.8 mm

Commit message: HW13 started
Parts:
- moved Q1 13.4 mm to (178.0, 87.2), turned to -90 degrees
- moved C5 8.93 mm to (163.2, 91.0), turned to 90 degrees
- moved C4 7.12 mm to (153.2, 91.0), turned to 90 degrees
- moved R17 6.49 mm to (185.0, 88.5)
- moved U2 1.79 mm to (158.2, 87.5), turned to 90 degrees
- moved R10 0.50 mm to (147.0, 81.0), turned to 180 degrees
Routing:
- net Net-(U4-QH'): track 0.00 -> 39.5 mm
- net Net-(Q1-B): track 27.8 -> 7.64 mm
- net Net-(U6-QH): track 40.8 -> 55.5 mm, vias 0 -> 1
- net P-P: track 59.2 -> 48.2 mm
- net +9V: track 104.9 -> 94.2 mm
- net GND: track 109.1 -> 116.1 mm
- net +5V: track 57.0 -> 59.2 mm
- net Net-(Q1-C): track 61.9 -> 62.8 mm
