File: HW13/HW13/HW13.kicad_sch (KiCad schematic)
At the start: 39 parts, among them J1 Barrel_Jack_MountingPin, U1 LM7805_TO220, U2 MC34063AP, U3 NE555P, U4 SC39-11SRWA, U5 SC39-11SRWA, U6 CD4026B, U7 CD4026B

Commit message: HW13 PCB done
Parts:
- U4, U5: footprint Display_7Segment:D1X8K -> Display_7Segment:Sx39-1xxxxx
Changed lines of the file:
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@@
 			)
 		)
-		(property "Footprint" "Display_7Segment:D1X8K"
+		(property "Footprint" "Display_7Segment:Sx39-1xxxxx"
 			(at 86.36 114.3 0)
 			(effects
@@
 		)
 		(instances
-			(project ""
+			(project "HW13"
 				(path "/2775b0cc-5ee2-4717-b361-3db89545ee8b"
 					(reference "U4")
@@
 			)
 		)
-		(property "Footprint" "Display_7Segment:D1X8K"
+		(property "Footprint" "Display_7Segment:Sx39-1xxxxx"
 			(at 163.83 114.3 0)
 			(effects
@@
 		)
 		(instances
-			(project ""
+			(project "HW13"
 				(path "/2775b0cc-5ee2-4717-b361-3db89545ee8b"
 					(reference "U6")
